File: hw/sch_pcb/EFMADC01.kicad_pcb (KiCad board)
At the start: 2 copper layers, 60.5 x 40.1 mm, 40 parts, among them J1 3.3-5V, J2 HEADER_2x01, J4 HEADER_2x01_PARALLEL, J5 HEADER_2x01_PARALLEL, J6 HEADER_2x01_PARALLEL, J7 HEADER_2x01_PARALLEL, J9 MCX, M1 RFShield_TwoPieces, M2 HOLE, M3 HOLE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

Commit message: Update to actual state
Parts:
- removed C7: 100nF, Capacitor_SMD:C_0805_2012Metric
- removed J2: HEADER_2x01, Mlab_Pin_Headers:Straight_2x01
- removed U1: ISL21080CIH315ZT, Package_TO_SOT_SMD:SOT-23
- added C13: 100nF, Capacitor_SMD:C_0805_2012Metric, B.Cu at (115.5, 81.8)
- added R8: 1k, Resistor_SMD:R_0805_2012Metric, B.Cu at (113.1, 86.4)
- added R9: 1k, Resistor_SMD:R_0805_2012Metric, B.Cu at (113.1, 89.8)
- added U5: OPA314, Package_TO_SOT_SMD:SOT-23-5, B.Cu at (112.4, 81.9)
- C2: value 100nF -> 10nF
- C4: value 1nF -> 10nF
- FID2: moved to F.Cu
- J1: value 3.3-5V -> 3.3 or 5V
- J9: moved to B.Cu
- R1: value 10M -> 270k
- R2: value 2k2 -> 3k3
- R3: value 10k -> 33k
- moved J1 122.6 mm to (69.3, 42.8)
- moved J4 122.6 mm to (69.3, 33.4)
- moved J6 122.6 mm to (69.3, 28.3)
- moved J7 122.6 mm to (69.3, 35.9)
- moved M2 122.6 mm to (20.8, 22.2)
- moved M3 122.6 mm to (71.6, 22.2)
- moved M4 122.6 mm to (20.8, 52.7)
- moved M5 122.6 mm to (71.6, 52.7)
- moved R7 122.6 mm to (65.1, 37.9)
- moved C6 122.6 mm to (65.7, 41.1)
- moved C8 122.6 mm to (65.7, 44.6)
- moved R4 122.6 mm to (65.3, 33.4)
- moved R5 122.6 mm to (65.3, 31.0)
- moved R6 122.6 mm to (65.3, 28.3)
- moved D2 122.6 mm to (73.5, 41.1)
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Connections:
- net Net-(J4-Pad1) renamed /SCK
- net Net-(J5-Pad1) renamed /SDO
- net Net-(J6-Pad1) renamed /SDI
- net Net-(J7-Pad1) renamed /CONV
- C11 pad 1: Net-(U4-V_{REF}) -> /ADC_REF
- U3 pad 2: Net-(U3-Vout) -> /ADC_REF
- U4 pad 10: Net-(U4-V_{REF}) -> /ADC_REF
Routing:
- net VCC: track 81.6 -> 98.9 mm, vias 0 -> 3
- net /ADC_REF: track 0.00 -> 13.8 mm
- net Net-(U4-V_{REF}): track 7.79 -> 0.00 mm
- net Net-(U5-+): track 0.00 -> 7.05 mm
- net Net-(J9-In): track 2.63 -> 9.64 mm
- net Net-(U4-SDI): track 16.7 -> 10.9 mm
- net GNDA: track 5.26 -> 10.3 mm, vias 0 -> 6
- net Net-(D1-A1): track 13.8 -> 18.7 mm
- net Net-(U4-CONV): track 19.0 -> 23.8 mm
- net /REF: track 23.8 -> 27.4 mm
- net Net-(U3-Vout): track 2.92 -> 0.00 mm
- net Net-(U4-SCK): track 11.8 -> 9.11 mm
- net GND: track 10.7 -> 8.15 mm, vias 22 -> 13
Other:
- board size 60.5 x 40.1 mm -> 130 x 130 mm
- board text removed: "Kaklik 2025"
- board text removed: "MLAB.cz"

Commit message: update layout
Parts:
- removed J4, J5, J6, J7: HEADER_2x01_PARALLEL, Mlab_Pin_Headers:Straight_2x01
- removed M2, M3, M4, M5: HOLE, Mlab_Mechanical:MountingHole_3mm
- added J1001: HEADER_2x10, Mlab_Pin_Headers:Straight_2x10, F.Cu at (131.1, 166.7)
- FID2: moved to B.Cu
- moved J1 150.3 mm to (152.4, 168.0)
- moved R6 145.3 mm to (124.8, 160.8), turned to -90 degrees
- moved R5 143.9 mm to (127.3, 160.8), turned to -90 degrees
- moved R4 142.9 mm to (130.0, 160.8), turned to -90 degrees
- moved C6 142.2 mm to (143.4, 160.1), turned to 0 degrees
- moved C8 141.2 mm to (143.3, 162.4), turned to 0 degrees
- moved R7 135.5 mm to (122.3, 160.8), turned to -90 degrees
- moved D2 134.4 mm to (140.7, 157.5), turned to 180 degrees
- moved FID1 4.44 mm to (90.2, 95.9)
- moved FID2 0.92 mm to (123.1, 63.7), turned to 0 degrees
Routing:
- net Net-(U4-SCK): track 9.11 -> 80.0 mm, vias 0 -> 2
- net Net-(U4-SDO): track 11.5 -> 77.8 mm, vias 0 -> 2
- net Net-(U4-CONV): track 23.8 -> 87.6 mm
- net Net-(U4-SDI): track 10.9 -> 74.5 mm, vias 0 -> 2
- net VCC: track 98.9 -> 146.0 mm
- net GND: track 8.15 -> 0.67 mm, vias 13 -> 170
- net /CONV: track 5.40 -> 3.77 mm
- net /SDO: track 4.47 -> 3.73 mm
- net /SDI: track 4.42 -> 3.75 mm
- net /SCK: track 4.42 -> 3.80 mm
Other:
- outline, holes or cut-outs redrawn
- board text added: "USTEFMADC01A"
- board text added: "VCC"
- board text removed: "+3.3V - +5V"
- board text removed: "ADC reference"
- board text removed: "ADC_REF"
- board text removed: "EFMADC01A"
- board text removed: "REF_out"
- board text removed: "Vcc"
