File: hw/sch_pcb/EFMADC01.kicad_sch (KiCad schematic)
At the start: 40 parts, among them J1 3.3-5V, J2 HEADER_2x01, J4 HEADER_2x01_PARALLEL, J5 HEADER_2x01_PARALLEL, J6 HEADER_2x01_PARALLEL, J7 HEADER_2x01_PARALLEL, J9 MCX, M1 RFShield_TwoPieces, M2 HOLE, M3 HOLE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

Commit message: Update to actual state
Parts:
- removed C7: 100nF, Capacitor_SMD:C_0805_2012Metric, symbol Device:C
- removed J2: HEADER_2x01, Mlab_Pin_Headers:Straight_2x01, symbol MLAB_HEADER:HEADER_2x01
- removed J4, J5, J6, J7: HEADER_2x01_PARALLEL, Mlab_Pin_Headers:Straight_2x01, symbol MLAB_HEADER:HEADER_2x01_PARALLEL
- removed U1: ISL21080CIH315ZT, Package_TO_SOT_SMD:SOT-23, symbol Reference_Voltage:ISL21070CIH320Z-TK
- added C13: 100nF, Capacitor_SMD:C_0805_2012Metric, symbol Device:C
- added J1001: HEADER_2x10, symbol MLAB_HEADER:HEADER_2x10
- added R8, R9: 1k, Resistor_SMD:R_0805_2012Metric, symbol Device:R
- added U5: OPA314, Package_TO_SOT_SMD:SOT-23-5, symbol Amplifier_Operational:OPA330xxDBV
- C2: value 100nF -> 10nF
- C4: value 1nF -> 10nF
- J1: value 3.3-5V -> 3.3 or 5V; now left out of the parts list
- R1: value 10M -> 270k
- R2: value 2k2 -> 3k3
- R3: value 10k -> 33k
Connections:
- net GND: now also J1001.19, J1001.20
- net GNDA: now also C13.1, R8.2, U5.2 (V-)
- net REF: now also U5.1, U5.4 (-)
- net VCC: now also C13.2, J1001.1, J1001.2, U5.5 (V+)
- net SCK: now reaches R4.2
- net SCK: now also J1001.11
- net ADC_REF: now reaches C11.1, U4.10 (V_{REF})
- net ADC_REF: now also U3.2 (Vout), R9.1
- net CONV: now reaches R7.2
- net CONV: now also J1001.17
- net SDO: now reaches R5.2
- net SDO: now also J1001.13
- net SDI: now reaches R6.2
- net SDI: now also J1001.15
- new net: R8.1, R9.2, U5.3 (+)
Other:
- note added: "Power input voltage depends on type of assembled ADC convertor. LTC1865 supports 5V, LTC1865L is 3v3."
- moved on the sheet: C1

Commit message: update layout
Parts:
- removed M2, M3, M4, M5: HOLE, Mlab_Mechanical:MountingHole_3mm, symbol MLAB_MECHANICAL:HOLE
- FID1, FID2: now not fitted
- J1001: footprint (none) -> Mlab_Pin_Headers:Straight_2x10
Other:
- note removed: "MOUNTING HOLES"
