File: hw/sch_pcb/USTEFMADC01.kicad_pcb (KiCad board)
At the start: 2 copper layers, 130 x 130 mm, 34 parts, among them J1 3.3 or 5V, J1001 HEADER_2x10, J9 MCX, M1 RFShield_TwoPieces, U2 OPA314, U3 ISL21080CIH330Z-TK, U4 LTC1865-MS, U5 OPA314

Commit message: solve DRC issues
Routing:
- net /ADC_REF: track 13.8 -> 12.7 mm
- net GND: vias 170 -> 180
Changed lines of the file:
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@@
 		(tags "capacitor")
 		(property "Reference" "C6"
-			(at -0.6604 -1.651 0)
+			(at 3.1 0.1 0)
 			(layer "B.SilkS")
 			(effects
@@
 	(segment
 		(start 109.44 90.266)
-		(end 110.575 90.266)
-		(width 0.45)
-		(layer "B.Cu")
-		(net 8)
-	)
-	(segment
-		(start 109.44 90.266)
 		(end 112.568 90.266)
 		(width 0.45)
@@
 	)
 	(via
-		(at 106.64 127)
+		(at 106.84 127.1)
 		(size 0.8)
 		(drill 0.4)
@@
 	)
 	(via
-		(at 106.64 115)
+		(at 106.84 115.3)
 		(size 0.8)
 		(drill 0.4)
@@
 	)
 	(via
+		(at 112.64 137.2)
+		(size 0.8)
+		(drill 0.4)
+		(layers "F.Cu" "B.Cu")
+		(free yes)
+		(net 13)
+	)
+	(via
 		(at 101.34 131.9)
 		(size 0.8)
@@
 	)
 	(via
-		(at 106.64 113)
+		(at 106.84 113.3)
 		(size 0.8)
 		(drill 0.4)
@@
 	)
 	(via
-		(at 106.64 129)
+		(at 106.84 129.1)
 		(size 0.8)
 		(drill 0.4)
@@
 	)
 	(via
+		(at 108.24 138.5)
+		(size 0.8)
+		(drill 0.4)
+		(layers "F.Cu" "B.Cu")
+		(free yes)
+		(net 13)
+	)
+	(via
 		(at 135.539495 150.699495)
 		(size 0.8)
@@
 	)
 	(via
+		(at 104.24 130)
+		(size 0.8)
+		(drill 0.4)
+		(layers "F.Cu" "B.Cu")
+		(free yes)
+		(net 13)
+	)
+	(via
 		(at 109.925786 150.185786)
 		(size 0.8)
@@
 	)
 	(via
-		(at 106.64 107)
+		(at 106.84 107.3)
+		(size 0.8)
+		(drill 0.4)
+		(layers "F.Cu" "B.Cu")
+		(free yes)
+		(net 13)
+	)
+	(via
+		(at 104.24 122)
 		(size 0.8)
 		(drill 0.4)
@@
 	)
 	(via
-		(at 106.64 121)
+		(at 106.84 121.1)
 		(size 0.8)
 		(drill 0.4)
@@
 	)
 	(via
-		(at 106.64 109)
+		(at 106.84 109.3)
 		(size 0.8)
 		(drill 0.4)
@@
 	)
 	(via
+		(at 104.24 126)
+		(size 0.8)
+		(drill 0.4)
+		(layers "F.Cu" "B.Cu")
+		(free yes)
+		(net 13)
+	)
+	(via
 		(at 118.411068 158.671068)
 		(size 0.8)
@@
 	)
 	(via
-		(at 113.04 106.5)
+		(at 96.84 113.6)
 		(size 0.8)
 		(drill 0.4)
@@
 	)
 	(via
-		(at 96.84 113.6)
+		(at 109.44 108.1)
 		(size 0.8)
 		(drill 0.4)
@@
 	)
 	(via
-		(at 109.44 108.1)
+		(at 104.24 132)
 		(size 0.8)
 		(drill 0.4)
@@
 	)
 	(via
-		(at 106.64 103)
+		(at 106.84 103.3)
 		(size 0.8)
 		(drill 0.4)
@@
 	)
 	(via
-		(at 106.64 125)
+		(at 106.84 125.1)
+		(size 0.8)
+		(drill 0.4)
+		(layers "F.Cu" "B.Cu")
+		(free yes)
+		(net 13)
+	)
+	(via
+		(at 104.24 120)
 		(size 0.8)
 		(drill 0.4)
@@
 	)
 	(via
+		(at 104.24 128)
+		(size 0.8)
+		(drill 0.4)
+		(layers "F.Cu" "B.Cu")
+		(free yes)
+		(net 13)
+	)
+	(via
 		(at 105.040505 140.500505)
 		(size 0.8)
@@
 	)
 	(via
-		(at 106.64 123)
+		(at 106.84 123.1)
 		(size 0.8)
 		(drill 0.4)
@@
 	)
 	(via
-		(at 113.04 108.5)
+		(at 113.04 109)
 		(size 0.8)
 		(drill 0.4)
@@
 	)
 	(via
-		(at 119.182641 154.642641)
+		(at 104.24 134)
 		(size 0.8)
 		(drill 0.4)
@@
 	)
 	(via
-		(at 101.34 125.9)
+		(at 119.182641 154.642641)
 		(size 0.8)
 		(drill 0.4)
@@
 	)
 	(via
-		(at 125.482136 165.742136)
+		(at 101.34 125.9)
 		(size 0.8)
 		(drill 0.4)
@@
 	)
 	(via
-		(at 106.64 105)
+		(at 106.84 105.3)
 		(size 0.8)
 		(drill 0.4)
@@
 	)
 	(via
-		(at 109.44 134.1)
+		(at 109.94 134.1)
 		(size 0.8)
 		(drill 0.4)
@@
 	)
 	(via
-		(at 106.64 111)
+		(at 106.84 111.3)
 		(size 0.8)
 		(drill 0.4)
@@
 	)
 	(via
+		(at 104.24 136)
+		(size 0.8)
+		(drill 0.4)
+		(layers "F.Cu" "B.Cu")
+		(free yes)
+		(net 13)
+	)
+	(via
 		(at 131.211068 155.471068)
 		(size 0.8)
@@
 	)
 	(via
-		(at 106.64 133)
+		(at 106.84 133.1)
 		(size 0.8)
 		(drill 0.4)
@@
 	)
 	(via
-		(at 106.64 135)
+		(at 106.84 135.1)
 		(size 0.8)
 		(drill 0.4)
@@
 	)
 	(via
-		(at 106.64 137)
+		(at 106.84 137.1)
 		(size 0.8)
 		(drill 0.4)
@@
 	)
 	(via
+		(at 104.24 124)
+		(size 0.8)
+		(drill 0.4)
+		(layers "F.Cu" "B.Cu")
+		(free yes)
+		(net 13)
+	)
+	(via
 		(at 127.054214 142.214214)
 		(size 0.8)
@@
 	)
 	(via
-		(at 106.64 131)
+		(at 109.64 139.9)
+		(size 0.8)
+		(drill 0.4)
+		(layers "F.Cu" "B.Cu")
+		(free yes)
+		(net 13)
+	)
+	(via
+		(at 106.84 131.1)
 		(size 0.8)
 		(drill 0.4)
