File: hw/sch_pcb/USTEFMADC01.kicad_pcb (KiCad board)
At the start: 2 copper layers, 130 x 130 mm, 34 parts, among them J1 3.3 or 5V, J1001 HEADER_2x10, J9 MCX, M1 RFShield_TwoPieces, U2 OPA314, U3 ISL21080CIH330Z-TK, U4 LTC1865-MS, U5 OPA314

Commit message: Upadte to version 01B, update actions
Parts:
- added J10: MCX, Connector_Coaxial:SMA_Amphenol_901-144_Vertical, F.Cu at (171.8, 140.2)
- added J11: MCX, Connector_Coaxial:SMA_Amphenol_901-144_Vertical, F.Cu at (90.4, 140.2)
Other:
- outline, holes or cut-outs redrawn
- board text added: "Mechanical"
- board text added: "SENSE"
- board text added: "USTEFMADC01B"
- board text removed: "USTEFMADC01A"

Commit message: solve issues
Other:
- board text added: "USTEFMADC01B 2026/05"
- board text removed: "USTEFMADC01B"
