File: hw/sch_pcb/USTEFMADC01.kicad_sch (KiCad schematic)
At the start: 34 parts, among them J1 3.3 or 5V, J1001 HEADER_2x10, J9 MCX, M1 RFShield_TwoPieces, U2 OPA314, U3 ISL21080CIH330Z-TK, U4 LTC1865-MS, U5 OPA314

Commit message: Upadte to version 01B, update actions
Parts:
- added J10, J11: MCX, Connector_Coaxial:SMA_Amphenol_901-144_Vertical, symbol Connector:Conn_Coaxial
Connections:
- net GND: now also J10.2 (Ext), J11.2 (Ext)
- no-connect marks 0 -> 14
Other:
- title: EFMADC01A -> EFMADC01B
